File: dc_switch.sch (KiCad schematic (older format))
At the start: 4 parts, among them J2 Conn_01x02_Male, J3 Conn_01x02_Male, Q1 Q_NMOS_GDS, Q2 Q_NMOS_GDS

Commit message: Associated footprints
Parts:
- J2, J3: footprint (none) -> Connector_Phoenix_MSTB:PhoenixContact_MSTBVA_2,5_2-G-5,08_1x02_P5.08mm_Vertical
- Q1, Q2: footprint (none) -> Package_TO_SOT_THT:TO-220F-3_Vertical
Changed lines of the file:
@@
 F 0 "J2" H 5872 3274 50  0000 R CNN
 F 1 "Conn_01x02_Male" H 5872 3183 50  0000 R CNN
-F 2 "" H 5900 3300 50  0001 C CNN
+F 2 "Connector_Phoenix_MSTB:PhoenixContact_MSTBVA_2,5_2-G-5,08_1x02_P5.08mm_Vertical" H 5900 3300 50  0001 C CNN
 F 3 "~" H 5900 3300 50  0001 C CNN
 	1    5900 3300
@@
 F 0 "Q1" H 4704 3396 50  0000 L CNN
 F 1 "Q_NMOS_GDS" H 4704 3305 50  0000 L CNN
-F 2 "" H 4700 3450 50  0001 C CNN
+F 2 "Package_TO_SOT_THT:TO-220F-3_Vertical" H 4700 3450 50  0001 C CNN
 F 3 "~" H 4500 3350 50  0001 C CNN
 	1    4500 3350
@@
 F 0 "Q2" H 4704 4646 50  0000 L CNN
 F 1 "Q_NMOS_GDS" H 4704 4555 50  0000 L CNN
-F 2 "" H 4700 4700 50  0001 C CNN
+F 2 "Package_TO_SOT_THT:TO-220F-3_Vertical" H 4700 4700 50  0001 C CNN
 F 3 "~" H 4500 4600 50  0001 C CNN
 	1    4500 4600
@@
 	6850 3300 7200 3300
 $Comp
-L power:GND #PWR?
+L power:GND #PWR0127
 U 1 1 5FF1DD74
 P 4600 3850
-F 0 "#PWR?" H 4600 3600 50  0001 C CNN
+F 0 "#PWR0127" H 4600 3600 50  0001 C CNN
 F 1 "GND" H 4605 3677 50  0000 C CNN
 F 2 "" H 4600 3850 50  0001 C CNN
@@
 Connection ~ 4600 3700
 $Comp
-L power:GND #PWR?
+L power:GND #PWR0128
 U 1 1 5FF1E8B0
 P 4600 5100
-F 0 "#PWR?" H 4600 4850 50  0001 C CNN
+F 0 "#PWR0128" H 4600 4850 50  0001 C CNN
 F 1 "GND" H 4605 4927 50  0000 C CNN
 F 2 "" H 4600 5100 50  0001 C CNN
@@
 F 0 "J3" H 5872 4524 50  0000 R CNN
 F 1 "Conn_01x02_Male" H 5872 4433 50  0000 R CNN
-F 2 "" H 5900 4550 50  0001 C CNN
+F 2 "Connector_Phoenix_MSTB:PhoenixContact_MSTBVA_2,5_2-G-5,08_1x02_P5.08mm_Vertical" H 5900 4550 50  0001 C CNN
 F 3 "~" H 5900 4550 50  0001 C CNN
 	1    5900 4550
